File: christmas-board.sch (KiCad schematic (older format))
At the start: 47 parts, among them J1 Conn_01x02_Female, Q1 Q_NPN_BCE, Q2 Q_NPN_BCE, Q3 Q_NPN_BCE, Q4 Q_NPN_BCE, Q5 Q_NPN_BCE, SW1 SW_Push, SW2 SW_Push, U1 595_SHIFT, U2 555

Commit message: assigned footprints to components
Parts:
- C1: footprint (none) -> Capacitor_THT:CP_Radial_D4.0mm_P1.50mm
- D1, D2, D3, D4, D5, D6, D7, D8: footprint (none) -> LED_THT:LED_D5.0mm
- J1: footprint (none) -> Connector_PinHeader_2.54mm:PinHeader_1x02_P2.54mm_Vertical
- Q1, Q2, Q3, Q4, Q5: footprint (none) -> Package_TO_SOT_THT:TO-92L_Inline
- R1, R10, R11, R12, R13, R14, R15, R16, R17, R18, R19, R2, R20, R21, R22, R23, R24, R25, R26, R27, R28, R3, R4, R5, R6, R7, R8, R9: footprint (none) -> Resistor_THT:R_Axial_DIN0204_L3.6mm_D1.6mm_P7.62mm_Horizontal
- SW1, SW2: footprint (none) -> Connector_PinHeader_2.54mm:PinHeader_2x01_P2.54mm_Vertical
- U1: footprint (none) -> Package_DIP:DIP-16_W7.62mm
- U2: footprint (none) -> Package_DIP:DIP-8_W7.62mm

Commit message: LED routing complete
Parts:
- removed Q1, Q2, Q3, Q4, Q5: Q_NPN_BCE, Package_TO_SOT_THT:TO-92L_Inline, symbol Device:Q_NPN_BCE
- added Q1, Q2, Q3, Q4, Q5: Q_NPN_CBE, Package_TO_SOT_THT:TO-92L_Inline, symbol Device:Q_NPN_CBE
Changed lines of the file:
@@
 $EndDescr
-$Comp
-L Device:Q_NPN_BCE Q2
-U 1 1 5BA47E0C
-P 3000 3400
-F 0 "Q2" H 3191 3446 50  0000 L CNN
-F 1 "Q_NPN_BCE" H 3191 3355 50  0000 L CNN
-F 2 "Package_TO_SOT_THT:TO-92L_Inline" H 3200 3500 50  0001 C CNN
-F 3 "~" H 3000 3400 50  0001 C CNN
-	1    3000 3400
-	1    0    0    -1
-$EndComp
 $Comp
 L Device:R R6
@@
 $EndComp
 $Comp
-L Device:Q_NPN_BCE Q1
-U 1 1 5BA4843D
-P 3000 2100
-F 0 "Q1" H 3191 2146 50  0000 L CNN
-F 1 "Q_NPN_BCE" H 3191 2055 50  0000 L CNN
-F 2 "Package_TO_SOT_THT:TO-92L_Inline" H 3200 2200 50  0001 C CNN
-F 3 "~" H 3000 2100 50  0001 C CNN
-	1    3000 2100
-	1    0    0    -1
-$EndComp
-$Comp
 L Device:R R5
 U 1 1 5BA48444
@@
 $EndComp
 $Comp
-L Device:Q_NPN_BCE Q3
-U 1 1 5BA48638
-P 6400 2700
-F 0 "Q3" H 6591 2746 50  0000 L CNN
-F 1 "Q_NPN_BCE" H 6591 2655 50  0000 L CNN
-F 2 "Package_TO_SOT_THT:TO-92L_Inline" H 6600 2800 50  0001 C CNN
-F 3 "~" H 6400 2700 50  0001 C CNN
-	1    6400 2700
-	1    0    0    -1
-$EndComp
-$Comp
 L Device:R R11
 U 1 1 5BA4863F
@@
 $EndComp
 $Comp
-L Device:Q_NPN_BCE Q4
-U 1 1 5BA488B5
-P 6400 4300
-F 0 "Q4" H 6591 4346 50  0000 L CNN
-F 1 "Q_NPN_BCE" H 6591 4255 50  0000 L CNN
-F 2 "Package_TO_SOT_THT:TO-92L_Inline" H 6600 4400 50  0001 C CNN
-F 3 "~" H 6400 4300 50  0001 C CNN
-	1    6400 4300
-	1    0    0    -1
-$EndComp
-$Comp
 L Device:R R12
 U 1 1 5BA488BC
@@
 	5100 4600 5100 4300
 Connection ~ 5100 4300
-$Comp
-L Device:Q_NPN_BCE Q5
-U 1 1 5BA4C44F
-P 9500 3500
-F 0 "Q5" H 9691 3546 50  0000 L CNN
-F 1 "Q_NPN_BCE" H 9691 3455 50  0000 L CNN
-F 2 "Package_TO_SOT_THT:TO-92L_Inline" H 9700 3600 50  0001 C CNN
-F 3 "~" H 9500 3500 50  0001 C CNN
-	1    9500 3500
-	1    0    0    -1
-$EndComp
 $Comp
 L Device:R R15
@@
 Wire Wire Line
 	11850 6550 11900 6550
+$Comp
+L Device:Q_NPN_CBE Q1
+U 1 1 5BB146CA
+P 3000 2100
+F 0 "Q1" H 3191 2146 50  0000 L CNN
+F 1 "Q_NPN_CBE" H 3191 2055 50  0000 L CNN
+F 2 "Package_TO_SOT_THT:TO-92L_Inline" H 3200 2200 50  0001 C CNN
+F 3 "~" H 3000 2100 50  0001 C CNN
+	1    3000 2100
+	1    0    0    -1
+$EndComp
+$Comp
+L Device:Q_NPN_CBE Q2
+U 1 1 5BB14DA8
+P 3000 3400
+F 0 "Q2" H 3191 3446 50  0000 L CNN
+F 1 "Q_NPN_CBE" H 3191 3355 50  0000 L CNN
+F 2 "Package_TO_SOT_THT:TO-92L_Inline" H 3200 3500 50  0001 C CNN
+F 3 "~" H 3000 3400 50  0001 C CNN
+	1    3000 3400
+	1    0    0    -1
+$EndComp
+$Comp
+L Device:Q_NPN_CBE Q3
+U 1 1 5BB14E2C
+P 6400 2700
+F 0 "Q3" H 6591 2746 50  0000 L CNN
+F 1 "Q_NPN_CBE" H 6591 2655 50  0000 L CNN
+F 2 "Package_TO_SOT_THT:TO-92L_Inline" H 6600 2800 50  0001 C CNN
+F 3 "~" H 6400 2700 50  0001 C CNN
+	1    6400 2700
+	1    0    0    -1
+$EndComp
+$Comp
+L Device:Q_NPN_CBE Q4
+U 1 1 5BB14EC0
+P 6400 4300
+F 0 "Q4" H 6591 4346 50  0000 L CNN
+F 1 "Q_NPN_CBE" H 6591 4255 50  0000 L CNN
+F 2 "Package_TO_SOT_THT:TO-92L_Inline" H 6600 4400 50  0001 C CNN
+F 3 "~" H 6400 4300 50  0001 C CNN
+	1    6400 4300
+	1    0    0    -1
+$EndComp
+$Comp
+L Device:Q_NPN_CBE Q5
+U 1 1 5BB14F4D
+P 9500 3500
+F 0 "Q5" H 9691 3546 50  0000 L CNN
+F 1 "Q_NPN_CBE" H 9691 3455 50  0000 L CNN
+F 2 "Package_TO_SOT_THT:TO-92L_Inline" H 9700 3600 50  0001 C CNN
+F 3 "~" H 9500 3500 50  0001 C CNN
+	1    9500 3500
+	1    0    0    -1
+$EndComp
 $EndSCHEMATC

Commit message: fix footprint on npn - swich to EBC ro CBE
Parts:
- removed Q1, Q2, Q3, Q4, Q5: Q_NPN_CBE, Package_TO_SOT_THT:TO-92L_Inline, symbol Device:Q_NPN_CBE
- added Q1, Q2, Q3, Q4, Q5: Q_NPN_EBC, Package_TO_SOT_THT:TO-92L_Inline, symbol Device:Q_NPN_EBC
Changed lines of the file:
@@
 	11850 6550 11900 6550
 $Comp
-L Device:Q_NPN_CBE Q1
-U 1 1 5BB146CA
+L Device:Q_NPN_EBC Q1
+U 1 1 5BB15809
 P 3000 2100
 F 0 "Q1" H 3191 2146 50  0000 L CNN
-F 1 "Q_NPN_CBE" H 3191 2055 50  0000 L CNN
+F 1 "Q_NPN_EBC" H 3191 2055 50  0000 L CNN
 F 2 "Package_TO_SOT_THT:TO-92L_Inline" H 3200 2200 50  0001 C CNN
 F 3 "~" H 3000 2100 50  0001 C CNN
@@
 $EndComp
 $Comp
-L Device:Q_NPN_CBE Q2
-U 1 1 5BB14DA8
+L Device:Q_NPN_EBC Q2
+U 1 1 5BB15A44
 P 3000 3400
 F 0 "Q2" H 3191 3446 50  0000 L CNN
-F 1 "Q_NPN_CBE" H 3191 3355 50  0000 L CNN
+F 1 "Q_NPN_EBC" H 3191 3355 50  0000 L CNN
 F 2 "Package_TO_SOT_THT:TO-92L_Inline" H 3200 3500 50  0001 C CNN
 F 3 "~" H 3000 3400 50  0001 C CNN
@@
 $EndComp
 $Comp
-L Device:Q_NPN_CBE Q3
-U 1 1 5BB14E2C
+L Device:Q_NPN_EBC Q3
+U 1 1 5BB15AF7
 P 6400 2700
 F 0 "Q3" H 6591 2746 50  0000 L CNN
-F 1 "Q_NPN_CBE" H 6591 2655 50  0000 L CNN
+F 1 "Q_NPN_EBC" H 6591 2655 50  0000 L CNN
 F 2 "Package_TO_SOT_THT:TO-92L_Inline" H 6600 2800 50  0001 C CNN
 F 3 "~" H 6400 2700 50  0001 C CNN
@@
 $EndComp
 $Comp
-L Device:Q_NPN_CBE Q4
-U 1 1 5BB14EC0
+L Device:Q_NPN_EBC Q4
+U 1 1 5BB15B96
 P 6400 4300
 F 0 "Q4" H 6591 4346 50  0000 L CNN
-F 1 "Q_NPN_CBE" H 6591 4255 50  0000 L CNN
+F 1 "Q_NPN_EBC" H 6591 4255 50  0000 L CNN
 F 2 "Package_TO_SOT_THT:TO-92L_Inline" H 6600 4400 50  0001 C CNN
 F 3 "~" H 6400 4300 50  0001 C CNN
@@
 $EndComp
 $Comp
-L Device:Q_NPN_CBE Q5
-U 1 1 5BB14F4D
+L Device:Q_NPN_EBC Q5
+U 1 1 5BB15C1E
 P 9500 3500
 F 0 "Q5" H 9691 3546 50  0000 L CNN
-F 1 "Q_NPN_CBE" H 9691 3455 50  0000 L CNN
+F 1 "Q_NPN_EBC" H 9691 3455 50  0000 L CNN
 F 2 "Package_TO_SOT_THT:TO-92L_Inline" H 9700 3600 50  0001 C CNN
 F 3 "~" H 9500 3500 50  0001 C CNN

Commit message: switch added, tracks updated
Parts:
- added SW3: SW_SPDT, Connector_PinHeader_2.54mm:PinHeader_1x03_P2.54mm_Vertical, symbol Switch:SW_SPDT
- SW1, SW2: footprint Connector_PinHeader_2.54mm:PinHeader_2x01_P2.54mm_Vertical -> christmas_board_footprint_lib:Tactile_Shallow_SW
Connections:
- wire segments 141 -> 144
- no-connect marks 1 -> 2
Changed lines of the file:
@@
 F 0 "SW2" H 13550 6235 50  0000 C CNN
 F 1 "SW_Push" H 13550 6144 50  0000 C CNN
-F 2 "Connector_PinHeader_2.54mm:PinHeader_2x01_P2.54mm_Vertical" H 13550 6150 50  0001 C CNN
+F 2 "christmas_board_footprint_lib:Tactile_Shallow_SW" H 13550 6150 50  0001 C CNN
 F 3 "" H 13550 6150 50  0001 C CNN
 	1    13550 5950
@@
 F 0 "SW1" H 13550 5685 50  0000 C CNN
 F 1 "SW_Push" H 13550 5594 50  0000 C CNN
-F 2 "Connector_PinHeader_2.54mm:PinHeader_2x01_P2.54mm_Vertical" H 13550 5600 50  0001 C CNN
+F 2 "christmas_board_footprint_lib:Tactile_Shallow_SW" H 13550 5600 50  0001 C CNN
 F 3 "" H 13550 5600 50  0001 C CNN
 	1    13550 5400
@@
 L Connector:Conn_01x02_Female J1
 U 1 1 5BADD2F0
-P 12100 6450
-F 0 "J1" H 12127 6426 50  0000 L CNN
-F 1 "Conn_01x02_Female" H 12127 6335 50  0000 L CNN
-F 2 "Connector_PinHeader_2.54mm:PinHeader_1x02_P2.54mm_Vertical" H 12100 6450 50  0001 C CNN
-F 3 "~" H 12100 6450 50  0001 C CNN
-	1    12100 6450
+P 12950 6450
+F 0 "J1" H 12977 6426 50  0000 L CNN
+F 1 "Conn_01x02_Female" H 12977 6335 50  0000 L CNN
+F 2 "Connector_PinHeader_2.54mm:PinHeader_1x02_P2.54mm_Vertical" H 12950 6450 50  0001 C CNN
+F 3 "~" H 12950 6450 50  0001 C CNN
+	1    12950 6450
 	1    0    0    -1
 $EndComp
@@
 Wire Wire Line
 	11850 6400 11850 6450
-Connection ~ 11850 6450
-Wire Wire Line
-	11850 6450 11900 6450
 $Comp
 L Device:CP C1
@@
 Connection ~ 11850 6550
 Wire Wire Line
-	11850 6550 11900 6550
+	11850 6550 12750 6550
 $Comp
 L Device:Q_NPN_EBC Q1
@@
 	1    0    0    -1
 $EndComp
+$Comp
+L Switch:SW_SPDT SW3
+U 1 1 5BB23971
+P 12350 6300
+F 0 "SW3" H 12350 6585 50  0000 C CNN
+F 1 "SW_SPDT" H 12350 6494 50  0000 C CNN
+F 2 "Connector_PinHeader_2.54mm:PinHeader_1x03_P2.54mm_Vertical" H 12350 6300 50  0001 C CNN
+F 3 "" H 12350 6300 50  0001 C CNN
+	1    12350 6300
+	1    0    0    -1
+$EndComp
+Wire Wire Line
+	11850 6450 12150 6450
+Wire Wire Line
+	12150 6450 12150 6300
+Connection ~ 11850 6450
+Wire Wire Line
+	12550 6400 12550 6450
+Wire Wire Line
+	12550 6450 12750 6450
+NoConn ~ 12550 6200
 $EndSCHEMATC
